Commit message: feat: added Gazebo simulation with LIDAR for Puzzlebot URDF

File: ros2_ws/src/puzzlebot_description/urdf/puzzlebot.urdf.xacro (robot description, xacro)
@@ -1,35 +1,41 @@
 <?xml version="1.0"?>
 <robot xmlns:xacro="http://ros.org/wiki/xacro" name="puzzlebot">
-    <xacro:property name="chassis_m"   value="0.8"/>
-    <xacro:property name="chassis_ixx" value="0.004"/>
-    <xacro:property name="wheel_m"     value="0.05"/>
-    <xacro:property name="wheel_ixx"   value="0.002"/>
+    <xacro:include filename="$(find puzzlebot_description)/urdf/puzzlebot_gazebo.xacro"/>
+    <xacro:include filename="$(find puzzlebot_description)/urdf/puzzlebot_ros2_control.xacro"/>
+    <xacro:property name="base_m"      value="1.2"/>
+    <xacro:property name="base_i"      value="0.001"/>
+    <xacro:property name="wheel_m"     value="0.053"/>
+    <xacro:property name="wheel_i"     value="0.001"/>
     <xacro:property name="wheel_rad"   value="0.05"/>
-    <xacro:property name="cas_rad"     value="0.0075"/>
-    <xacro:property name="dummy_m"     value="0.001"/>
-    <xacro:property name="dummy_ixx"   value="1.0e-6"/>
-    <xacro:macro name="dummy_inertial">
-        <inertial>
-            <origin xyz="0 0 0" rpy="0 0 0"/>
-            <mass value="${dummy_m}"/>
-            <inertia ixx="${dummy_ixx}" iyy="${dummy_ixx}" izz="${dummy_ixx}" ixy="0.0" ixz="0.0" iyz="0.0"/>
-        </inertial>
-    </xacro:macro>
-    <link name="base_footprint">
-        <xacro:dummy_inertial/>
-    </link>
+    <xacro:property name="wheel_x"     value="0.098"/>
+    <xacro:property name="wheel_y"     value="-0.038"/>
+    <xacro:property name="caster_m"    value="1.0E-06"/>
+    <xacro:property name="caster_i"    value="1.0E-10"/>
+    <xacro:property name="caster_rad"  value="0.0075"/>
+    <xacro:property name="blue_rgba"       value="0.0 0.5 1.0 1.0"/>
+    <xacro:property name="dark_grey_rgba"  value="0.2 0.2 0.2 1.0"/>
+    <link name="base_footprint"/>
     <link name="base_link">
         <inertial>
             <origin xyz="0 0 0" rpy="0 0 0"/>
-            <mass value="${chassis_m}"/>
-            <inertia ixx="${chassis_ixx}" iyy="${chassis_ixx}" izz="${chassis_ixx}" ixy="0.0" ixz="0.0" iyz="0.0"/>
+            <mass value="${base_m}"/>
+            <inertia ixx="${base_i}" ixy="0.0" ixz="0.0"
+                     iyy="${base_i}" iyz="0.0"
+                     izz="${base_i}"/>
         </inertial>
         <visual>
             <origin xyz="0 0 0" rpy="1.5708 0 0"/>
-            <geometry><mesh filename="package://puzzlebot_description/meshes/chassis.stl"/></geometry>
+            <geometry>
+                <mesh filename="package://puzzlebot_description/meshes/chassis.stl"/>
+            </geometry>
+            <material name="chassis_color">
+                <color rgba="${blue_rgba}"/>
+            </material>
         </visual>
         <collision>
             <origin xyz="0 0 0" rpy="1.5708 0 0"/>
-            <geometry><mesh filename="package://puzzlebot_description/meshes/chassis.stl"/></geometry>
+            <geometry>
+                <mesh filename="package://puzzlebot_description/meshes/chassis.stl"/>
+            </geometry>
         </collision>
     </link>
@@ -43,12 +49,22 @@
             <origin xyz="0 0 0" rpy="0 0 0"/>
             <mass value="${wheel_m}"/>
-            <inertia ixx="${wheel_ixx}" iyy="${wheel_ixx}" izz="${wheel_ixx}" ixy="0.0" ixz="0.0" iyz="0.0"/>
+            <inertia ixx="${wheel_i}" ixy="0.0" ixz="0.0"
+                     iyy="${wheel_i}" iyz="0.0"
+                     izz="${wheel_i}"/>
         </inertial>
         <visual>
             <origin xyz="0 0 0" rpy="0 -1.5708 0"/>
-            <geometry><mesh filename="package://puzzlebot_description/meshes/wheel.stl"/></geometry>
+            <geometry>
+                <mesh filename="package://puzzlebot_description/meshes/wheel.stl"/>
+            </geometry>
+            <material name="wheel_color">
+                <color rgba="${blue_rgba}"/>
+            </material>
         </visual>
         <collision>
-            <geometry><sphere radius="${wheel_rad}"/></geometry>
+            <origin xyz="0 0 0" rpy="0 0 0"/>
+            <geometry>
+                <sphere radius="${wheel_rad}"/>
+            </geometry>
         </collision>
     </link>
@@ -57,5 +73,5 @@
         <child link="wheel_right_link"/>
         <axis xyz="1 0 0"/>
-        <origin xyz="0.098 -0.038 0" rpy="0 0 0"/>
+        <origin xyz="${wheel_x} ${wheel_y} 0" rpy="0 0 0"/>
     </joint>
     <link name="wheel_left_link">
@@ -63,12 +79,22 @@
             <origin xyz="0 0 0" rpy="0 0 0"/>
             <mass value="${wheel_m}"/>
-            <inertia ixx="${wheel_ixx}" iyy="${wheel_ixx}" izz="${wheel_ixx}" ixy="0.0" ixz="0.0" iyz="0.0"/>
+            <inertia ixx="${wheel_i}" ixy="0.0" ixz="0.0"
+                     iyy="${wheel_i}" iyz="0.0"
+                     izz="${wheel_i}"/>
         </inertial>
         <visual>
             <origin xyz="0 0 0" rpy="0 1.5708 0"/>
-            <geometry><mesh filename="package://puzzlebot_description/meshes/wheel.stl"/></geometry>
+            <geometry>
+                <mesh filename="package://puzzlebot_description/meshes/wheel.stl"/>
+            </geometry>
+            <material name="wheel_color">
+                <color rgba="${blue_rgba}"/>
+            </material>
         </visual>
         <collision>
-            <geometry><sphere radius="${wheel_rad}"/></geometry>
+            <origin xyz="0 0 0" rpy="0 0 0"/>
+            <geometry>
+                <sphere radius="${wheel_rad}"/>
+            </geometry>
         </collision>
     </link>
@@ -77,10 +103,19 @@
         <child link="wheel_left_link"/>
         <axis xyz="1 0 0"/>
-        <origin xyz="-0.098 -0.038 0" rpy="0 0 0"/>
+        <origin xyz="-${wheel_x} ${wheel_y} 0" rpy="0 0 0"/>
     </joint>
     <link name="caster_link">
-        <xacro:dummy_inertial/>
+        <inertial>
+            <origin xyz="0 0 0" rpy="0 0 0"/>
+            <mass value="${caster_m}"/>
+            <inertia ixx="${caster_i}" ixy="0.0" ixz="0.0"
+                     iyy="${caster_i}" iyz="0.0"
+                     izz="${caster_i}"/>
+        </inertial>
         <collision>
-            <geometry><sphere radius="${cas_rad}"/></geometry>
+            <origin xyz="0 0 0" rpy="0 0 0"/>
+            <geometry>
+                <sphere radius="${caster_rad}"/>
+            </geometry>
         </collision>
     </link>
@@ -88,13 +123,19 @@
         <parent link="base_footprint"/>
         <child link="caster_link"/>
-        <origin xyz="0 0.095 0" rpy="0 0 0"/>
+        <origin xyz="0 0.095 0.0081" rpy="0 0 0"/>
     </joint>
     <link name="laser_link">
-        <xacro:dummy_inertial/>
         <visual>
-            <geometry><mesh filename="package://puzzlebot_description/meshes/laser_link.STL"/></geometry>
+            <geometry>
+                <mesh filename="package://puzzlebot_description/meshes/laser_link.stl"/>
+            </geometry>
+            <material name="laser_color">
+                <color rgba="${dark_grey_rgba}"/>
+            </material>
         </visual>
         <collision>
-            <geometry><mesh filename="package://puzzlebot_description/meshes/laser_link.STL"/></geometry>
+            <geometry>
+                <mesh filename="package://puzzlebot_description/meshes/laser_link.stl"/>
+            </geometry>
         </collision>
     </link>

Commit message: fix: fixed URDF axis

File: ros2_ws/src/puzzlebot_description/urdf/puzzlebot.urdf.xacro (robot description, xacro)
@@ -8,9 +8,10 @@
     <xacro:property name="wheel_i"     value="0.001"/>
     <xacro:property name="wheel_rad"   value="0.05"/>
-    <xacro:property name="wheel_x"     value="0.098"/>
-    <xacro:property name="wheel_y"     value="-0.038"/>
+    <xacro:property name="wheel_x"     value="0.038"/>
+    <xacro:property name="wheel_y"     value="0.098"/>
     <xacro:property name="caster_m"    value="1.0E-06"/>
     <xacro:property name="caster_i"    value="1.0E-10"/>
     <xacro:property name="caster_rad"  value="0.0075"/>
+    <xacro:property name="caster_x"    value="-0.095"/>
     <xacro:property name="blue_rgba"       value="0.0 0.5 1.0 1.0"/>
     <xacro:property name="dark_grey_rgba"  value="0.2 0.2 0.2 1.0"/>
@@ -25,5 +26,5 @@
         </inertial>
         <visual>
-            <origin xyz="0 0 0" rpy="1.5708 0 0"/>
+            <origin xyz="0 0 0" rpy="1.5708 0 1.5708"/>
             <geometry>
                 <mesh filename="package://puzzlebot_description/meshes/chassis.stl"/>
@@ -34,5 +35,5 @@
         </visual>
         <collision>
-            <origin xyz="0 0 0" rpy="1.5708 0 0"/>
+            <origin xyz="0 0 0" rpy="1.5708 0 1.5708"/>
             <geometry>
                 <mesh filename="package://puzzlebot_description/meshes/chassis.stl"/>
@@ -54,5 +55,5 @@
         </inertial>
         <visual>
-            <origin xyz="0 0 0" rpy="0 -1.5708 0"/>
+            <origin xyz="0 0 0" rpy="0 -1.5708 1.5708"/>
             <geometry>
                 <mesh filename="package://puzzlebot_description/meshes/wheel.stl"/>
@@ -72,6 +73,6 @@
         <parent link="base_link"/>
         <child link="wheel_right_link"/>
-        <axis xyz="1 0 0"/>
-        <origin xyz="${wheel_x} ${wheel_y} 0" rpy="0 0 0"/>
+        <axis xyz="0 1 0"/>
+        <origin xyz="${wheel_x} -${wheel_y} 0" rpy="0 0 0"/>
     </joint>
     <link name="wheel_left_link">
@@ -84,5 +85,5 @@
         </inertial>
         <visual>
-            <origin xyz="0 0 0" rpy="0 1.5708 0"/>
+            <origin xyz="0 0 0" rpy="0 1.5708 1.5708"/>
             <geometry>
                 <mesh filename="package://puzzlebot_description/meshes/wheel.stl"/>
@@ -102,6 +103,6 @@
         <parent link="base_link"/>
         <child link="wheel_left_link"/>
-        <axis xyz="1 0 0"/>
-        <origin xyz="-${wheel_x} ${wheel_y} 0" rpy="0 0 0"/>
+        <axis xyz="0 1 0"/>
+        <origin xyz="${wheel_x} ${wheel_y} 0" rpy="0 0 0"/>
     </joint>
     <link name="caster_link">
@@ -123,8 +124,9 @@
         <parent link="base_footprint"/>
         <child link="caster_link"/>
-        <origin xyz="0 0.095 0.0081" rpy="0 0 0"/>
+        <origin xyz="${caster_x} 0 0.0081" rpy="0 0 0"/>
     </joint>
     <link name="laser_link">
         <visual>
+            <origin xyz="0 0 0" rpy="0 0 3.14159"/>
             <geometry>
                 <mesh filename="package://puzzlebot_description/meshes/laser_link.stl"/>
@@ -143,5 +145,5 @@
         <parent link="base_link" />
         <child link="laser_link" />
-        <origin xyz="-0.005 -0.002 0.12" rpy="0 0 3.14" />
+        <origin xyz="0.05 0.0 0.12" rpy="0 0 3.14159" />
     </joint>
 </robot>

Commit message: fix: modified xyz origin of LIDAR to resemble real life Puzzlebot

File: ros2_ws/src/puzzlebot_description/urdf/puzzlebot.urdf.xacro (robot description, xacro)
@@ -145,5 +145,5 @@
         <parent link="base_link" />
         <child link="laser_link" />
-        <origin xyz="0.05 0.0 0.12" rpy="0 0 3.14159" />
+        <origin xyz="0.038 0.0 0.115" rpy="0 0 3.14159" />
     </joint>
 </robot>

Commit message: feat: add camera simulation

File: ros2_ws/src/puzzlebot_description/urdf/puzzlebot.urdf.xacro (robot description, xacro)
@@ -137,4 +137,5 @@
         </visual>
         <collision>
+            <origin xyz="0 0 0" rpy="0 0 3.14159"/>
             <geometry>
                 <mesh filename="package://puzzlebot_description/meshes/laser_link.stl"/>
@@ -147,3 +148,25 @@
         <origin xyz="0.038 0.0 0.115" rpy="0 0 3.14159" />
     </joint>
+    <link name="camera_link">
+        <visual>
+            <origin xyz="0 0 0" rpy="1.5708 0 1.5708"/>
+            <geometry>
+                <mesh filename="package://puzzlebot_description/meshes/camera.stl"/>
+            </geometry>
+            <material name="camera_color">
+                <color rgba="${blue_rgba}"/>
+            </material>
+        </visual>
+    </link>
+    <joint name="camera_joint" type="fixed">
+        <parent link="base_link"/>
+        <child link="camera_link"/>
+        <origin xyz="0.1 0.0 0.05" rpy="0 0 0"/>
+    </joint>
+    <link name="camera_optical_link"/>
+    <joint name="camera_optical_joint" type="fixed">
+        <parent link="camera_link"/>
+        <child link="camera_optical_link"/>
+        <origin xyz="0 0 0" rpy="-1.5708 0 -1.5708"/>
+    </joint>
 </robot>

File: ros2_ws/src/puzzlebot_description/urdf/puzzlebot_gazebo.xacro (robot description, xacro)
@@ -66,3 +66,43 @@
         </sensor>
     </gazebo>
+    <gazebo reference="camera_link">
+        <sensor name="camera" type="camera">
+            <always_on>true</always_on>
+            <visualize>true</visualize>
+            <update_rate>30</update_rate>
+            <camera>
+                <camera_info_topic>camera_info</camera_info_topic>
+                <horizontal_fov>1.089</horizontal_fov>
+                <image>
+                    <format>R8G8B8</format>
+                    <width>640</width>
+                    <height>480</height>
+                </image>
+                <clip>
+                    <near>0.05</near>
+                    <far>8.0</far>
+                </clip>
+                <lens>
+                    <intrinsics>
+                        <fx>277.1</fx> <!-- Focal length X -->
+                        <fy>277.1</fy> <!-- Focal length Y -->
+                        <cx>320.5</cx> <!-- Principal point X -->
+                        <cy>240.5</cy> <!-- Principal point Y -->
+                        <s>0</s>        <!-- Skew -->
+                    </intrinsics>
+                </lens>
+                <distortion>
+                    <k1>0.0</k1>
+                    <k2>0.0</k2>
+                    <k3>0.0</k3>
+                    <p1>0.0</p1>
+                    <p2>0.0</p2>
+                    <center>0.5 0.5</center>
+                </distortion>
+                <!-- ============================================== -->
+            </camera>
+            <topic>image_raw</topic>
+            <gz_frame_id>camera_link_optical</gz_frame_id>
+        </sensor>
+    </gazebo>
 </robot>

Commit message: feat: optimized simulation (slow af)

File: ros2_ws/src/puzzlebot_description/urdf/puzzlebot.urdf.xacro (robot description, xacro)
@@ -16,4 +16,5 @@
     <xacro:property name="blue_rgba"       value="0.0 0.5 1.0 1.0"/>
     <xacro:property name="dark_grey_rgba"  value="0.2 0.2 0.2 1.0"/>
+    <!-- BASE -->
     <link name="base_footprint"/>
     <link name="base_link">
@@ -26,5 +27,5 @@
         </inertial>
         <visual>
-            <origin xyz="0 0 0" rpy="1.5708 0 1.5708"/>
+            <origin xyz="0 0 0" rpy="${pi/2} 0 ${pi/2}"/>
             <geometry>
                 <mesh filename="package://puzzlebot_description/meshes/chassis.stl"/>
@@ -35,5 +36,5 @@
         </visual>
         <collision>
-            <origin xyz="0 0 0" rpy="1.5708 0 1.5708"/>
+            <origin xyz="0 0 0" rpy="${pi/2} 0 ${pi/2}"/>
             <geometry>
                 <mesh filename="package://puzzlebot_description/meshes/chassis.stl"/>
@@ -46,4 +47,5 @@
         <origin xyz="0 0 0.05" rpy="0 0 0"/>
     </joint>
+    <!-- RIGHT WHEEL -->
     <link name="wheel_right_link">
         <inertial>
@@ -55,5 +57,5 @@
         </inertial>
         <visual>
-            <origin xyz="0 0 0" rpy="0 -1.5708 1.5708"/>
+            <origin xyz="0 0 0" rpy="0 ${-pi/2} ${pi/2}"/>
             <geometry>
                 <mesh filename="package://puzzlebot_description/meshes/wheel.stl"/>
@@ -76,4 +78,5 @@
         <origin xyz="${wheel_x} -${wheel_y} 0" rpy="0 0 0"/>
     </joint>
+    <!-- LEFT WHEEL -->
     <link name="wheel_left_link">
         <inertial>
@@ -85,5 +88,5 @@
         </inertial>
         <visual>
-            <origin xyz="0 0 0" rpy="0 1.5708 1.5708"/>
+            <origin xyz="0 0 0" rpy="0 ${pi/2} ${pi/2}"/>
             <geometry>
                 <mesh filename="package://puzzlebot_description/meshes/wheel.stl"/>
@@ -106,4 +109,5 @@
         <origin xyz="${wheel_x} ${wheel_y} 0" rpy="0 0 0"/>
     </joint>
+    <!-- CASTER -->
     <link name="caster_link">
         <inertial>
@@ -126,7 +130,8 @@
         <origin xyz="${caster_x} 0 0.0081" rpy="0 0 0"/>
     </joint>
+    <!-- LASER -->
     <link name="laser_link">
         <visual>
-            <origin xyz="0 0 0" rpy="0 0 3.14159"/>
+            <origin xyz="0 0 0" rpy="0 0 ${pi}"/>
             <geometry>
                 <mesh filename="package://puzzlebot_description/meshes/laser_link.stl"/>
@@ -136,19 +141,14 @@
             </material>
         </visual>
-        <collision>
-            <origin xyz="0 0 0" rpy="0 0 3.14159"/>
-            <geometry>
-                <mesh filename="package://puzzlebot_description/meshes/laser_link.stl"/>
-            </geometry>
-        </collision>
     </link>
     <joint name="laser_joint" type="fixed">
         <parent link="base_link" />
         <child link="laser_link" />
-        <origin xyz="0.038 0.0 0.115" rpy="0 0 3.14159" />
+        <origin xyz="0.038 0.0 0.115" rpy="0 0 ${pi}" />
     </joint>
+    <!-- CAMERA -->
     <link name="camera_link">
         <visual>
-            <origin xyz="0 0 0" rpy="1.5708 0 1.5708"/>
+            <origin xyz="0 0 0" rpy="${pi/2} 0 ${pi/2}"/>
             <geometry>
                 <mesh filename="package://puzzlebot_description/meshes/camera.stl"/>
@@ -164,9 +164,10 @@
         <origin xyz="0.1 0.0 0.05" rpy="0 0 0"/>
     </joint>
+    <!-- CAMERA OPTICAL -->
     <link name="camera_optical_link"/>
     <joint name="camera_optical_joint" type="fixed">
         <parent link="camera_link"/>
         <child link="camera_optical_link"/>
-        <origin xyz="0 0 0" rpy="-1.5708 0 -1.5708"/>
+        <origin xyz="0 0 0" rpy="${-pi/2} 0 ${-pi/2}"/>
     </joint>
 </robot>

File: ros2_ws/src/puzzlebot_description/urdf/puzzlebot_gazebo.xacro (robot description, xacro)
@@ -73,5 +73,5 @@
             <always_on>true</always_on>
             <visualize>true</visualize>
-            <update_rate>30</update_rate>
+            <update_rate>10</update_rate>
             <camera>
                 <camera_info_topic>camera_info</camera_info_topic>

Commit message: fix: renamed laser_link to link so it works with real robot; feat: added twist mux between joystick and PID; feat: added launch file for real robot, everything works alright!

File: ros2_ws/src/puzzlebot_description/urdf/puzzlebot.urdf.xacro (robot description, xacro)
@@ -131,5 +131,5 @@
     </joint>
     <!-- LASER -->
-    <link name="laser_link">
+    <link name="laser">
         <visual>
             <origin xyz="0 0 0" rpy="0 0 ${pi}"/>
@@ -144,5 +144,5 @@
     <joint name="laser_joint" type="fixed">
         <parent link="base_link" />
-        <child link="laser_link" />
+        <child link="laser" />
         <origin xyz="0.038 0.0 0.115" rpy="0 0 ${pi}" />
     </joint>

File: ros2_ws/src/puzzlebot_description/urdf/puzzlebot_gazebo.xacro (robot description, xacro)
@@ -40,5 +40,5 @@
     https://cdn.robotshop.com/media/r/rpk/rb-rpk-03/pdf/ld108_slamtec_rplidar_datasheet_a1m8_v3.0_en.pdf?_gl=1*69cea1*_gcl_au*MTg0MzU2MTI3Ni4xNzc3NTA5NzA1*_ga*MTk3OTA5Nzg3MS4xNzc3NTA5NzA1*_ga_FXHVC4EYRV*czE3Nzc1MDk3MDQkbzEkZzAkdDE3Nzc1MDk3MDQkajYwJGwwJGgw
     -->
-    <gazebo reference="laser_link">
+    <gazebo reference="laser">
         <sensor name="lidar" type="gpu_lidar">
             <always_on>true</always_on>
@@ -46,5 +46,5 @@
             <update_rate>5.5</update_rate>
             <topic>scan</topic>
-            <gz_frame_id>laser_link</gz_frame_id>
+            <gz_frame_id>laser</gz_frame_id>
             <lidar>
                 <scan>
